Commit message: kind of working

File: my_dual_robot_cell/my_dual_robot_cell_description/urdf/my_dual_robot_cell_macro.xacro (robot description, xacro)
@@ -30,5 +30,5 @@
     headless_mode:=false
     ">
-    <joint name="table_base_joint" type="fixed">
+     <!-- <joint name="table_base_joint" type="fixed">
       <xacro:insert_block name="origin" />
       <parent link="${parent}" />
@@ -48,6 +48,6 @@
         <origin rpy="0 0 0" xyz="0.75 0.5 -1"/>
       </collision>
-    </link>
-    <link name="monitor">
+    </link> -->
+   <!-- <link name="monitor">
       <visual>
         <geometry>
@@ -60,14 +60,14 @@
         </geometry>
       </collision>
-    </link>
-    <joint name="base_to_monitor" type="fixed">
-      <parent link="table"/>
+    </link>  -->
+    <!-- <joint name="base_to_monitor" type="fixed">-->
+      <!-- <parent link="table"/>
       <child link="monitor"/>
       <origin xyz="0.2 0.6 0"/>
-    </joint>
-    <material name="white">
+    </joint>  -->
+    <!-- <material name="white">
       <color rgba="1 1 1 1"/>
-    </material>
-    <link name="wall">
+    </material> -->
+    <!-- <link name="wall">
       <visual>
         <geometry>
@@ -85,7 +85,7 @@
       <child link="wall"/>
       <origin xyz="1.25 1.5 0.5"/>
-    </joint>
+    </joint> -->
     <!--Creates the mounts to attach the robots to the table-->
-    <link name="alice_robot_mount"/>
+    <!-- <link name="alice_robot_mount"/>
     <joint name="base_to_alice_robot_mount" type="fixed">
       <parent link="table"/>
@@ -98,10 +98,10 @@
       <child link="bob_robot_mount"/>
       <origin xyz="1.0 0.85 0" rpy="0 0 ${pi}" />
-    </joint>
-    <!--Creates the 1st Robot-->
+    </joint> -->
+    Creates the 1st Robot
     <xacro:ur_robot
       name="alice"
       tf_prefix="alice_"
-      parent="alice_robot_mount"
+      parent="world"
       joint_limits_parameters_file="${alice_joint_limits_parameters_file}"
       kinematics_parameters_file="${alice_kinematics_parameters_file}"
@@ -124,5 +124,5 @@
       name="bob"
       tf_prefix="bob_"
-      parent="bob_robot_mount"
+      parent="world"
       joint_limits_parameters_file="${bob_joint_limits_parameters_file}"
       kinematics_parameters_file="${bob_kinematics_parameters_file}"
@@ -139,5 +139,5 @@
       headless_mode="${headless_mode}"
     >
-      <origin xyz="0 0 0" rpy="0 0 0" />
+      <origin xyz="0 1 0" rpy="0 0 0" />
     </xacro:ur_robot>
   </xacro:macro>

Commit message: working an tested on real hardware

File: my_dual_robot_cell/my_dual_robot_cell_description/urdf/my_dual_robot_cell_macro.xacro (robot description, xacro)
@@ -139,5 +139,5 @@
       headless_mode="${headless_mode}"
     >
-      <origin xyz="0 1 0" rpy="0 0 0" />
+      <origin xyz="0 3 0" rpy="0 0 0" />
     </xacro:ur_robot>
   </xacro:macro>
