Commit message: changes robot names

File: my_dual_robot_cell/my_dual_robot_cell_control/urdf/my_dual_robot_cell_controlled.urdf.xacro (robot description, xacro)
@@ -7,28 +7,28 @@
   <!-- <xacro:include filename="$(find ur_description)/urdf/ur.ros2_control.xacro" /> -->
   <!--We need to specify the arguments used for parametrizing our description-->
-  <xacro:arg name="alice_ur_type" default="ur3" />
-  <xacro:arg name="alice_joint_limits_parameters_file" default="$(find ur_description)/config/$(arg alice_ur_type)/joint_limits.yaml" />
-  <xacro:arg name="alice_kinematics_parameters_file" default="$(find ur_description)/config/$(arg alice_ur_type)/default_kinematics.yaml" />
-  <xacro:arg name="alice_physical_parameters_file" default="$(find ur_description)/config/$(arg alice_ur_type)/physical_parameters.yaml" />
-  <xacro:arg name="alice_visual_parameters_file" default="$(find ur_description)/config/$(arg alice_ur_type)/visual_parameters.yaml" />
-  <xacro:arg name="bob_ur_type" default="ur3" />
-  <xacro:arg name="bob_joint_limits_parameters_file" default="$(find ur_description)/config/$(arg bob_ur_type)/joint_limits.yaml" />
-  <xacro:arg name="bob_kinematics_parameters_file" default="$(find ur_description)/config/$(arg bob_ur_type)/default_kinematics.yaml" />
-  <xacro:arg name="bob_physical_parameters_file" default="$(find ur_description)/config/$(arg bob_ur_type)/physical_parameters.yaml" />
-  <xacro:arg name="bob_visual_parameters_file" default="$(find ur_description)/config/$(arg bob_ur_type)/visual_parameters.yaml" />
-  <xacro:arg name="alice_use_mock_hardware" default="false" />
-  <xacro:arg name="alice_mock_sensor_commands" default="false" />
-  <xacro:arg name="alice_robot_ip" default="192.168.56.101" />
-  <xacro:arg name="alice_reverse_port" default="50006" />
-  <xacro:arg name="alice_script_sender_port" default="50007" />
-  <xacro:arg name="alice_script_command_port" default="50010" />
-  <xacro:arg name="alice_trajectory_port" default="50009" />
-  <xacro:arg name="bob_use_mock_hardware" default="false" />
-  <xacro:arg name="bob_mock_sensor_commands" default="false" />
-  <xacro:arg name="bob_robot_ip" default="192.168.56.102" />
-  <xacro:arg name="bob_reverse_port" default="50001" />
-  <xacro:arg name="bob_script_sender_port" default="50002" />
-  <xacro:arg name="bob_script_command_port" default="50004" />
-  <xacro:arg name="bob_trajectory_port" default="50003" />
+  <xacro:arg name="robot2_ur_type" default="ur3" />
+  <xacro:arg name="robot2_joint_limits_parameters_file" default="$(find ur_description)/config/$(arg robot2_ur_type)/joint_limits.yaml" />
+  <xacro:arg name="robot2_kinematics_parameters_file" default="$(find ur_description)/config/$(arg robot2_ur_type)/default_kinematics.yaml" />
+  <xacro:arg name="robot2_physical_parameters_file" default="$(find ur_description)/config/$(arg robot2_ur_type)/physical_parameters.yaml" />
+  <xacro:arg name="robot2_visual_parameters_file" default="$(find ur_description)/config/$(arg robot2_ur_type)/visual_parameters.yaml" />
+  <xacro:arg name="robot1_ur_type" default="ur3" />
+  <xacro:arg name="robot1_joint_limits_parameters_file" default="$(find ur_description)/config/$(arg robot1_ur_type)/joint_limits.yaml" />
+  <xacro:arg name="robot1_kinematics_parameters_file" default="$(find ur_description)/config/$(arg robot1_ur_type)/default_kinematics.yaml" />
+  <xacro:arg name="robot1_physical_parameters_file" default="$(find ur_description)/config/$(arg robot1_ur_type)/physical_parameters.yaml" />
+  <xacro:arg name="robot1_visual_parameters_file" default="$(find ur_description)/config/$(arg robot1_ur_type)/visual_parameters.yaml" />
+  <xacro:arg name="robot2_use_mock_hardware" default="false" />
+  <xacro:arg name="robot2_mock_sensor_commands" default="false" />
+  <xacro:arg name="robot2_robot_ip" default="192.168.56.101" />
+  <xacro:arg name="robot2_reverse_port" default="50006" />
+  <xacro:arg name="robot2_script_sender_port" default="50007" />
+  <xacro:arg name="robot2_script_command_port" default="50010" />
+  <xacro:arg name="robot2_trajectory_port" default="50009" />
+  <xacro:arg name="robot1_use_mock_hardware" default="false" />
+  <xacro:arg name="robot1_mock_sensor_commands" default="false" />
+  <xacro:arg name="robot1_robot_ip" default="192.168.56.102" />
+  <xacro:arg name="robot1_reverse_port" default="50001" />
+  <xacro:arg name="robot1_script_sender_port" default="50002" />
+  <xacro:arg name="robot1_script_command_port" default="50004" />
+  <xacro:arg name="robot1_trajectory_port" default="50003" />
   <xacro:arg name="headless_mode" default="false" />
   <xacro:arg name="ur_script_filename" default="$(find ur_client_library)/resources/external_control.urscript" />
@@ -38,24 +38,24 @@
   <xacro:my_dual_robot_cell
     parent="world"
-    alice_ur_type="$(arg alice_ur_type)"
-    alice_joint_limits_parameters_file="$(arg alice_joint_limits_parameters_file)"
-    alice_kinematics_parameters_file="$(arg alice_kinematics_parameters_file)"
-    alice_physical_parameters_file="$(arg alice_physical_parameters_file)"
-    alice_visual_parameters_file="$(arg alice_visual_parameters_file)"
-    alice_robot_ip="$(arg alice_robot_ip)"
-    alice_reverse_port="$(arg alice_reverse_port)"
-    alice_script_sender_port ="$(arg alice_script_sender_port)"
-    alice_script_command_port="$(arg alice_script_command_port)"
-    alice_trajectory_port="$(arg alice_trajectory_port)"
-    bob_ur_type="$(arg bob_ur_type)"
-    bob_joint_limits_parameters_file="$(arg bob_joint_limits_parameters_file)"
-    bob_kinematics_parameters_file="$(arg bob_kinematics_parameters_file)"
-    bob_physical_parameters_file="$(arg bob_physical_parameters_file)"
-    bob_visual_parameters_file="$(arg bob_visual_parameters_file)"
-    bob_robot_ip="$(arg bob_robot_ip)"
-    bob_reverse_port="$(arg bob_reverse_port)"
-    bob_script_sender_port ="$(arg bob_script_sender_port)"
-    bob_script_command_port="$(arg bob_script_command_port)"
-    bob_trajectory_port="$(arg bob_trajectory_port)"
+    robot2_ur_type="$(arg robot2_ur_type)"
+    robot2_joint_limits_parameters_file="$(arg robot2_joint_limits_parameters_file)"
+    robot2_kinematics_parameters_file="$(arg robot2_kinematics_parameters_file)"
+    robot2_physical_parameters_file="$(arg robot2_physical_parameters_file)"
+    robot2_visual_parameters_file="$(arg robot2_visual_parameters_file)"
+    robot2_robot_ip="$(arg robot2_robot_ip)"
+    robot2_reverse_port="$(arg robot2_reverse_port)"
+    robot2_script_sender_port ="$(arg robot2_script_sender_port)"
+    robot2_script_command_port="$(arg robot2_script_command_port)"
+    robot2_trajectory_port="$(arg robot2_trajectory_port)"
+    robot1_ur_type="$(arg robot1_ur_type)"
+    robot1_joint_limits_parameters_file="$(arg robot1_joint_limits_parameters_file)"
+    robot1_kinematics_parameters_file="$(arg robot1_kinematics_parameters_file)"
+    robot1_physical_parameters_file="$(arg robot1_physical_parameters_file)"
+    robot1_visual_parameters_file="$(arg robot1_visual_parameters_file)"
+    robot1_robot_ip="$(arg robot1_robot_ip)"
+    robot1_reverse_port="$(arg robot1_reverse_port)"
+    robot1_script_sender_port ="$(arg robot1_script_sender_port)"
+    robot1_script_command_port="$(arg robot1_script_command_port)"
+    robot1_trajectory_port="$(arg robot1_trajectory_port)"
     script_filename="$(arg ur_script_filename)"
     output_recipe_filename="$(arg ur_output_recipe_filename)"
@@ -66,28 +66,28 @@
   </xacro:my_dual_robot_cell>
   <!-- <xacro:ur_ros2_control
-    name="alice"
-    tf_prefix="alice_"
-    robot_ip="$(arg alice_robot_ip)"
+    name="robot2"
+    tf_prefix="robot2_"
+    robot_ip="$(arg robot2_robot_ip)"
     script_filename="$(arg ur_script_filename)"
     output_recipe_filename="$(arg ur_output_recipe_filename)"
     input_recipe_filename="$(arg ur_input_recipe_filename)"
     headless_mode="$(arg headless_mode)"
-    reverse_port="$(arg alice_reverse_port)"
-    script_sender_port="$(arg alice_script_sender_port)"
-    script_command_port="$(arg alice_script_command_port)"
-    trajectory_port="$(arg alice_trajectory_port)"
+    reverse_port="$(arg robot2_reverse_port)"
+    script_sender_port="$(arg robot2_script_sender_port)"
+    script_command_port="$(arg robot2_script_command_port)"
+    trajectory_port="$(arg robot2_trajectory_port)"
   />
   <xacro:ur_ros2_control
-    name="bob"
-    tf_prefix="bob_"
-    robot_ip="$(arg bob_robot_ip)"
+    name="robot1"
+    tf_prefix="robot1_"
+    robot_ip="$(arg robot1_robot_ip)"
     script_filename="$(arg ur_script_filename)"
     output_recipe_filename="$(arg ur_output_recipe_filename)"
     input_recipe_filename="$(arg ur_input_recipe_filename)"
     headless_mode="$(arg headless_mode)"
-    reverse_port="$(arg bob_reverse_port)"
-    script_sender_port="$(arg bob_script_sender_port)"
-    script_command_port="$(arg bob_script_command_port)"
-    trajectory_port="$(arg bob_trajectory_port)"
+    reverse_port="$(arg robot1_reverse_port)"
+    script_sender_port="$(arg robot1_script_sender_port)"
+    script_command_port="$(arg robot1_script_command_port)"
+    trajectory_port="$(arg robot1_trajectory_port)"
   />
   <xacro:ur_ros2_control
@@ -102,7 +102,7 @@
         output_recipe_filename="${output_recipe_filename}"
         input_recipe_filename="${input_recipe_filename}"
-        tf_prefix="bob_"
+        tf_prefix="robot1_"
         hash_kinematics="${kinematics_hash}"
-        robot_ip="$(arg bob_robot_ip)"
+        robot_ip="$(arg robot1_robot_ip)"
         use_tool_communication="${use_tool_communication}"
         tool_voltage="${tool_voltage}"

File: my_dual_robot_cell/my_dual_robot_cell_description/urdf/my_dual_robot_cell.urdf.xacro (robot description, xacro)
@@ -2,28 +2,28 @@
 <robot name="my_dual_robot_cell" xmlns:xacro="http://ros.org/wiki/xacro">
   <xacro:include filename="$(find my_dual_robot_cell_description)/urdf/my_dual_robot_cell_macro.xacro"/>
-  <xacro:arg name="alice_ur_type" default="ur3"/>
-  <xacro:arg name="alice_joint_limits_parameters_file" default="$(find ur_description)/config/$(arg alice_ur_type)/joint_limits.yaml"/>
-  <xacro:arg name="alice_kinematics_parameters_file" default="$(find ur_description)/config/$(arg alice_ur_type)/default_kinematics.yaml"/>
-  <xacro:arg name="alice_physical_parameters_file" default="$(find ur_description)/config/$(arg alice_ur_type)/physical_parameters.yaml"/>
-  <xacro:arg name="alice_visual_parameters_file" default="$(find ur_description)/config/$(arg alice_ur_type)/visual_parameters.yaml"/>
-  <xacro:arg name="bob_ur_type" default="ur3"/>
-  <xacro:arg name="bob_joint_limits_parameters_file" default="$(find ur_description)/config/$(arg bob_ur_type)/joint_limits.yaml"/>
-  <xacro:arg name="bob_kinematics_parameters_file" default="$(find ur_description)/config/$(arg bob_ur_type)/default_kinematics.yaml"/>
-  <xacro:arg name="bob_physical_parameters_file" default="$(find ur_description)/config/$(arg bob_ur_type)/physical_parameters.yaml"/>
-  <xacro:arg name="bob_visual_parameters_file" default="$(find ur_description)/config/$(arg bob_ur_type)/visual_parameters.yaml"/>
+  <xacro:arg name="robot2_ur_type" default="ur3"/>
+  <xacro:arg name="robot2_joint_limits_parameters_file" default="$(find ur_description)/config/$(arg robot2_ur_type)/joint_limits.yaml"/>
+  <xacro:arg name="robot2_kinematics_parameters_file" default="$(find ur_description)/config/$(arg robot2_ur_type)/default_kinematics.yaml"/>
+  <xacro:arg name="robot2_physical_parameters_file" default="$(find ur_description)/config/$(arg robot2_ur_type)/physical_parameters.yaml"/>
+  <xacro:arg name="robot2_visual_parameters_file" default="$(find ur_description)/config/$(arg robot2_ur_type)/visual_parameters.yaml"/>
+  <xacro:arg name="robot1_ur_type" default="ur3"/>
+  <xacro:arg name="robot1_joint_limits_parameters_file" default="$(find ur_description)/config/$(arg robot1_ur_type)/joint_limits.yaml"/>
+  <xacro:arg name="robot1_kinematics_parameters_file" default="$(find ur_description)/config/$(arg robot1_ur_type)/default_kinematics.yaml"/>
+  <xacro:arg name="robot1_physical_parameters_file" default="$(find ur_description)/config/$(arg robot1_ur_type)/physical_parameters.yaml"/>
+  <xacro:arg name="robot1_visual_parameters_file" default="$(find ur_description)/config/$(arg robot1_ur_type)/visual_parameters.yaml"/>
   <link name="world"/>
   <!--This will create the scene where the robots are located in-->
   <xacro:my_dual_robot_cell
     parent="world"
-    alice_ur_type="$(arg alice_ur_type)"
-    alice_joint_limits_parameters_file="$(arg alice_joint_limits_parameters_file)"
-    alice_kinematics_parameters_file="$(arg alice_kinematics_parameters_file)"
-    alice_physical_parameters_file="$(arg alice_physical_parameters_file)"
-    alice_visual_parameters_file="$(arg alice_visual_parameters_file)"
-    bob_ur_type="$(arg bob_ur_type)"
-    bob_joint_limits_parameters_file="$(arg bob_joint_limits_parameters_file)"
-    bob_kinematics_parameters_file="$(arg bob_kinematics_parameters_file)"
-    bob_physical_parameters_file="$(arg bob_physical_parameters_file)"
-    bob_visual_parameters_file="$(arg bob_visual_parameters_file)"
+    robot2_ur_type="$(arg robot2_ur_type)"
+    robot2_joint_limits_parameters_file="$(arg robot2_joint_limits_parameters_file)"
+    robot2_kinematics_parameters_file="$(arg robot2_kinematics_parameters_file)"
+    robot2_physical_parameters_file="$(arg robot2_physical_parameters_file)"
+    robot2_visual_parameters_file="$(arg robot2_visual_parameters_file)"
+    robot1_ur_type="$(arg robot1_ur_type)"
+    robot1_joint_limits_parameters_file="$(arg robot1_joint_limits_parameters_file)"
+    robot1_kinematics_parameters_file="$(arg robot1_kinematics_parameters_file)"
+    robot1_physical_parameters_file="$(arg robot1_physical_parameters_file)"
+    robot1_visual_parameters_file="$(arg robot1_visual_parameters_file)"
     >
       <origin xyz="0 0 1" rpy="0 0 0" />

File: my_dual_robot_cell/my_dual_robot_cell_description/urdf/my_dual_robot_cell_macro.xacro (robot description, xacro)
@@ -5,24 +5,24 @@
     parent
     *origin
-    alice_ur_type
-    alice_joint_limits_parameters_file
-    alice_kinematics_parameters_file
-    alice_physical_parameters_file
-    alice_visual_parameters_file
-    alice_robot_ip
-    alice_reverse_port
-    alice_script_sender_port
-    alice_script_command_port
-    alice_trajectory_port
-    bob_ur_type
-    bob_joint_limits_parameters_file
-    bob_kinematics_parameters_file
-    bob_physical_parameters_file
-    bob_visual_parameters_file
-    bob_robot_ip
-    bob_reverse_port
-    bob_script_sender_port
-    bob_script_command_port
-    bob_trajectory_port
+    robot2_ur_type
+    robot2_joint_limits_parameters_file
+    robot2_kinematics_parameters_file
+    robot2_physical_parameters_file
+    robot2_visual_parameters_file
+    robot2_robot_ip
+    robot2_reverse_port
+    robot2_script_sender_port
+    robot2_script_command_port
+    robot2_trajectory_port
+    robot1_ur_type
+    robot1_joint_limits_parameters_file
+    robot1_kinematics_parameters_file
+    robot1_physical_parameters_file
+    robot1_visual_parameters_file
+    robot1_robot_ip
+    robot1_reverse_port
+    robot1_script_sender_port
+    robot1_script_command_port
+    robot1_trajectory_port
     script_filename
     output_recipe_filename
@@ -87,30 +87,30 @@
     </joint> -->
     <!--Creates the mounts to attach the robots to the table-->
-    <!-- <link name="alice_robot_mount"/>
-    <joint name="base_to_alice_robot_mount" type="fixed">
+    <!-- <link name="robot2_robot_mount"/>
+    <joint name="base_to_robot2_robot_mount" type="fixed">
       <parent link="table"/>
-      <child link="alice_robot_mount"/>
+      <child link="robot2_robot_mount"/>
       <origin xyz="0.3 0.85 0" rpy="0 0 ${pi}" />
     </joint>
-    <link name="bob_robot_mount"/>
-    <joint name="base_to_bob_robot_mount" type="fixed">
+    <link name="robot1_robot_mount"/>
+    <joint name="base_to_robot1_robot_mount" type="fixed">
       <parent link="table"/>
-      <child link="bob_robot_mount"/>
+      <child link="robot1_robot_mount"/>
       <origin xyz="1.0 0.85 0" rpy="0 0 ${pi}" />
     </joint> -->
     Creates the 1st Robot
     <xacro:ur_robot
-      name="alice"
-      tf_prefix="alice_"
+      name="robot2"
+      tf_prefix="robot2_"
       parent="world"
-      joint_limits_parameters_file="${alice_joint_limits_parameters_file}"
-      kinematics_parameters_file="${alice_kinematics_parameters_file}"
-      physical_parameters_file="${alice_physical_parameters_file}"
-      visual_parameters_file="${alice_visual_parameters_file}"
-      robot_ip="${alice_robot_ip}"
-      reverse_port="${alice_reverse_port}"
-      script_sender_port="${alice_script_sender_port}"
-      script_command_port="${alice_script_command_port}"
-      trajectory_port="${alice_trajectory_port}"
+      joint_limits_parameters_file="${robot2_joint_limits_parameters_file}"
+      kinematics_parameters_file="${robot2_kinematics_parameters_file}"
+      physical_parameters_file="${robot2_physical_parameters_file}"
+      visual_parameters_file="${robot2_visual_parameters_file}"
+      robot_ip="${robot2_robot_ip}"
+      reverse_port="${robot2_reverse_port}"
+      script_sender_port="${robot2_script_sender_port}"
+      script_command_port="${robot2_script_command_port}"
+      trajectory_port="${robot2_trajectory_port}"
       script_filename="${script_filename}"
       output_recipe_filename="${output_recipe_filename}"
@@ -122,16 +122,16 @@
     <!--Creates the 2nd Robot-->
     <xacro:ur_robot
-      name="bob"
-      tf_prefix="bob_"
+      name="robot1"
+      tf_prefix="robot1_"
       parent="world"
-      joint_limits_parameters_file="${bob_joint_limits_parameters_file}"
-      kinematics_parameters_file="${bob_kinematics_parameters_file}"
-      physical_parameters_file="${bob_physical_parameters_file}"
-      visual_parameters_file="${bob_visual_parameters_file}"
-      robot_ip="${bob_robot_ip}"
-      reverse_port="${bob_reverse_port}"
-      script_sender_port="${bob_script_sender_port}"
-      script_command_port="${bob_script_command_port}"
-      trajectory_port="${bob_trajectory_port}"
+      joint_limits_parameters_file="${robot1_joint_limits_parameters_file}"
+      kinematics_parameters_file="${robot1_kinematics_parameters_file}"
+      physical_parameters_file="${robot1_physical_parameters_file}"
+      visual_parameters_file="${robot1_visual_parameters_file}"
+      robot_ip="${robot1_robot_ip}"
+      reverse_port="${robot1_reverse_port}"
+      script_sender_port="${robot1_script_sender_port}"
+      script_command_port="${robot1_script_command_port}"
+      trajectory_port="${robot1_trajectory_port}"
       script_filename="${script_filename}"
       output_recipe_filename="${output_recipe_filename}"
